File: I2C-7-Segment-Backpack-dot56inch.brd (EAGLE design)
At the start: 45.7 x 33 mm, 20 parts, among them J1 4P-SMD-2.0-90D, U1 AS1115

Commit message: Rev C
Other:
- board text added: "I2C 7 SEGMENT BKPK .56" (Rev C)"
- board text added: "dcity.org"
- board text removed: "I2C 7 SEGMENT BKPK .56" (Rev B)"
- board text removed: "wht.io"
Changed lines of the file:
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@@
 <?xml version="1.0" encoding="utf-8"?>
 <!DOCTYPE eagle SYSTEM "eagle.dtd">
-<eagle version="7.5.0">
+<eagle version="9.1.3">
 <drawing>
 <settings>
 <setting alwaysvectorfont="no"/>
+<setting keepoldvectorfont="yes"/>
 <setting verticaltext="up"/>
 </settings>
@@
 <text x="7.62" y="29.21" size="0.889" layer="21" font="vector" ratio="15">SJ3 CLOSED = 01h</text>
 <text x="24.13" y="27.94" size="0.889" layer="21" font="vector" ratio="15">DO NOT CLOSE BOTH</text>
-<text x="35.56" y="1.27" size="0.889" layer="22" font="vector" ratio="15" rot="MR0">I2C 7 SEGMENT BKPK .56" (Rev B)</text>
+<text x="35.56" y="1.27" size="0.889" layer="22" font="vector" ratio="15" rot="MR0">I2C 7 SEGMENT BKPK .56" (Rev C)</text>
 <text x="28.067" y="6.35" size="0.889" layer="21" font="vector" ratio="15" rot="R180">LED1</text>
 <text x="19.812" y="6.35" size="0.889" layer="22" font="vector" ratio="15" rot="MR180">LED1</text>
@@
 <rectangle x1="27.432" y1="19.812" x2="29.845" y2="21.082" layer="43"/>
 <rectangle x1="31.496" y1="22.098" x2="33.147" y2="23.241" layer="43"/>
-<text x="35.941" y="24.765" size="1.778" layer="21" font="vector" ratio="10">wht.io</text>
-<text x="27.178" y="2.794" size="1.778" layer="22" font="vector" ratio="10" rot="MR0">wht.io</text>
+<text x="32.7406" y="25.4254" size="1.778" layer="21" font="vector" ratio="10">dcity.org</text>
+<text x="27.178" y="2.794" size="1.778" layer="22" font="vector" ratio="10" rot="MR0">dcity.org</text>
 </plain>
 <attributes>
@@
 <param name="dpMaxLengthDifference" value="10mm"/>
 <param name="dpGapFactor" value="2.5"/>
-<param name="checkGrid" value="0"/>
 <param name="checkAngle" value="1"/>
 <param name="checkFont" value="1"/>
 <param name="checkRestrict" value="1"/>
+<param name="checkStop" value="0"/>
+<param name="checkValues" value="0"/>
+<param name="checkNames" value="1"/>
+<param name="checkWireStubs" value="1"/>
+<param name="checkPolygonWidth" value="0"/>
 <param name="useDiameter" value="13"/>
 <param name="maxErrors" value="50"/>
@@
 </signal>
 </signals>
+<mfgpreviewcolors>
+<mfgpreviewcolor name="soldermaskcolor" color="0xC8008000"/>
+<mfgpreviewcolor name="silkscreencolor" color="0xFFFEFEFE"/>
+<mfgpreviewcolor name="backgroundcolor" color="0xFF282828"/>
+<mfgpreviewcolor name="coppercolor" color="0xFFFFBF00"/>
+<mfgpreviewcolor name="substratecolor" color="0xFF786E46"/>
+</mfgpreviewcolors>
 </board>
 </drawing>

Commit message: Rev D
Parts:
- added J3: QWIIC_RIGHT_ANGLE, 0:JST04_1MM_RA
- J1: value 4P-SMD-2.0-90D -> QWIIC_RIGHT_ANGLE; device 0:HW4-SMD-2.0-90D -> 0:JST04_1MM_RA
- moved J1 6.35 mm to (40.6, 20.3), turned to 90 degrees
- moved J2 2.54 mm to (34.3, 20.3)
Connections:
- net GND: now also J1.1, J3.1; no longer J1.4
- net SCL: now also J1.4, J3.4; no longer J1.1
- net SDA: now also J1.3, J3.3; no longer J1.2
- net VCC: now also J1.2, J3.2; no longer J1.3
Routing:
- net N$8: track 43.1 -> 80.4 mm
- net N$6: track 51.8 -> 32.8 mm, vias 2 -> 4
- net SDA: track 58.1 -> 75.4 mm
- net VCC: track 70.1 -> 84.9 mm
- net N$5: track 36.3 -> 50.2 mm, vias 0 -> 2
- net SCL: track 61.1 -> 74.1 mm
- net N$4: track 33.3 -> 38.3 mm
- net GND: track 12.8 -> 13.3 mm, vias 3 -> 5
Other:
- board text added: "0.56 inch LED - (Rev D)"
- board text added: "I2C 7 SEGMENT BKPK .56" (Rev D)"
- board text removed: "0.56 inch LED - (Rev B)"
- board text removed: "I2C 7 SEGMENT BKPK .56" (Rev C)"
