File: I2C-7-Segment-Backpack-dot56inch.sch (EAGLE design)
At the start: 20 parts, among them J1 4P-SMD-2.0-90D, U1 AS1115

Commit message: Rev D
Parts:
- added J3: QWIIC_RIGHT_ANGLE, 0:QWIIC_CONNECTORJS-1MM
- J1: value 4P-SMD-2.0-90D -> QWIIC_RIGHT_ANGLE; device 0:GROVE-CONNECTOR-SMD-90D(4+2P-2.0) -> 0:QWIIC_CONNECTORJS-1MM
Connections:
- net GND: now also J1.1, J3.1; no longer J1.4
- net SCL: now also J1.4, J3.4; no longer J1.1
- net SDA: now also J1.3, J3.3; no longer J1.2
- net VCC: now also J1.2, J3.2; no longer J1.3
